Commit message: Fix PointCloud tf error

File: urdf/camera/camera.gazebo.xacro (robot description, xacro)
@@ -1,5 +1,5 @@
 <?xml version="1.0"?>
 <robot name="csi_camera" xmlns:xacro="http://ros.org/wiki/xacro">
-  <xacro:macro name="camera_gazebo" params="camera_name camera_link robot_namespace">
+  <xacro:macro name="camera_gazebo" params="camera_name camera_link robot_namespace robotdescription_namespace">
     <link name="${camera_link}_tf_origin" />
     <joint name="${camera_link}_tf_joint" type="fixed">
@@ -37,5 +37,5 @@
           <imageTopicName>image_raw</imageTopicName>
           <cameraInfoTopicName>camera_info</cameraInfoTopicName>
-          <frameName>${camera_link}_tf_origin</frameName>
+          <frameName>${robotdescription_namespace}${camera_link}_tf_origin</frameName>
           <hackBaseline>0.0</hackBaseline>
           <distortionK1>0.0</distortionK1>

File: urdf/jnmouse.urdf.xacro (robot description, xacro)
@@ -5,4 +5,5 @@
        xmlns:interface="http://playerstage.sourceforge.net/gazebo/xmlschema/#interface"
        xmlns:xacro="http://ros.org/wiki/xacro">
+  <xacro:arg name="camera_namespace" default="stereo_camera" />
   <xacro:include filename="$(find jnmouse_description)/urdf/common.xacro" />
   <xacro:include filename="$(find jnmouse_description)/urdf/body/body.urdf.xacro" />
@@ -48,6 +49,10 @@
   <xacro:lightsensor_gazebo prefix="lf" base_rad="0" rad_range="0.3" min_range="0.01" max_range="0.6" robot_namespace="raspimouse_on_gazebo" />
   <!-- Cameras -->
-  <xacro:camera_gazebo camera_name="right" camera_link="right_camera_link" robot_namespace="stereo_camera" />
-  <xacro:camera_gazebo camera_name="left" camera_link="left_camera_link" robot_namespace="stereo_camera" />
+  <xacro:camera_gazebo camera_name="right" camera_link="right_camera_link"
+    robot_namespace="$(arg camera_namespace)"
+    robotdescription_namespace="/" />
+  <xacro:camera_gazebo camera_name="left" camera_link="left_camera_link"
+    robot_namespace="$(arg camera_namespace)"
+    robotdescription_namespace="/" />
   <!-- DiffDriveController -->
   <gazebo>
