Commit message: Fix tread parameter
ref: https://github.com/rt-net/raspimouse_description/issues/33

File: urdf/common.xacro (robot description, xacro)
@@ -4,5 +4,5 @@
   <xacro:property name="wheel_length" value="0.010" />
   <xacro:property name="wheel_mass" value="0.0113" />
-  <xacro:property name="wheel_separation" value="0.0935" />
+  <xacro:property name="wheel_separation" value="0.0925" />
   <!-- PROPERTY LIST -->
   <!-- All units in m-kg-s-radians unit system -->
